Commit message: fixing xacro for publishing the joint state correctly

File: ackermann_vehicle_description/urdf/em_3905.urdf.xacro (robot description, xacro)
@@ -200,5 +200,7 @@
     <transmission name="${lr_prefix}_${fr_prefix}_shock_trans">
       <type>transmission_interface/SimpleTransmission</type>
-      <joint name="${lr_prefix}_${fr_prefix}_shock"/>
+      <joint name="${lr_prefix}_${fr_prefix}_shock">
+        <hardwareInterface>EffortJointInterface</hardwareInterface>
+      </joint>
       <actuator name="${lr_prefix}_${fr_prefix}_shock_act">
         <hardwareInterface>EffortJointInterface</hardwareInterface>
@@ -223,5 +225,7 @@
     <transmission name="${lr_prefix}_${fr_prefix}_axle_trans">
       <type>transmission_interface/SimpleTransmission</type>
-      <joint name="${lr_prefix}_${fr_prefix}_axle"/>
+      <joint name="${lr_prefix}_${fr_prefix}_axle">
+        <hardwareInterface>EffortJointInterface</hardwareInterface>
+      </joint>
       <actuator name="${lr_prefix}_${fr_prefix}_axle_act">
         <hardwareInterface>EffortJointInterface</hardwareInterface>
@@ -275,5 +279,7 @@
     <transmission name="${lr_prefix}_steering_trans">
       <type>transmission_interface/SimpleTransmission</type>
-      <joint name="${lr_prefix}_steering_joint"/>
+      <joint name="${lr_prefix}_steering_joint">
+        <hardwareInterface>EffortJointInterface</hardwareInterface>
+      </joint>
       <actuator name="${lr_prefix}_steering_act">
         <hardwareInterface>EffortJointInterface</hardwareInterface>
